Commit message: Config Changes for Luffy
Various changes to get code working on Luffy. Also start to trying to fix moveit loading the collision model too slowly

File: xacro/gummi.srdf.xacro (robot description, xacro)
@@ -18,5 +18,4 @@
         <xacro:group_right_arm_ee />
     </group>
-    <xacro:group_right_gripper_ee />
     <!--GROUP STATES: Purpose: Define a named state for a particular group, in terms of joint values. This is useful to define states like 'folded arms'-->
     <group_state name="default" group="right_arm">
@@ -24,5 +23,4 @@
       <xacro:group_state_right_arm_ee />
     </group_state>
-    <xacro:end_effector_ee />
     <xacro:virtual_joints_base />
     <xacro:disable_collisions_base />

File: xacro/gummi_description_base.urdf.xacro (robot description, xacro)
@@ -23,5 +23,5 @@
       <geometry>
         <mesh
-          filename="package://gummi_base_$(env ROS_GUMMI_BASE)/meshes/base_Link.stl" />
+          filename="package://gummi_base_$(env ROS_GUMMI_BASE)/meshes/base_Link1.stl" />
       </geometry>
       <material
@@ -37,5 +37,5 @@
       <geometry>
         <mesh
-          filename="package://gummi_base_$(env ROS_GUMMI_BASE)/meshes/base_Link.stl" />
+          filename="package://gummi_base_$(env ROS_GUMMI_BASE)/meshes/base_Link1.stl" />
       </geometry>
     </collision>
@@ -144,5 +144,5 @@
     <origin
       xyz="0 -0.065 0.1265"
-      rpy="1.57 0 0" />
+      rpy="-1.57 3.16 0" />
     <parent
       link="shoulder_preroll" />
@@ -150,5 +150,5 @@
       link="shoulder" />
     <axis
-      xyz="0 -1 0" />
+      xyz="0 0 -1" />
     <limit
       lower="-0.95"
@@ -201,6 +201,6 @@
     type="revolute">
     <origin
-      xyz="-0.024 -0.17679 8.6827E-05"
-      rpy="0 0 0" />
+      xyz="-0.019 0 -0.054"
+      rpy="-1.57 0 1.57" />
     <parent
       link="shoulder" />
@@ -208,5 +208,5 @@
       link="upperarm_preroll" />
     <axis
-      xyz="-1 0 0" />
+      xyz="0 0 -1" />
     <limit
       lower="-0.15"
@@ -259,6 +259,6 @@
     type="revolute">
     <origin
-      xyz="0.056992 -0.010088 -0.035587"
-      rpy="0 0 0" />
+      xyz="-0.0355 0.00999 0.0145"
+      rpy="-1.57 0 -1.57" />
     <parent
       link="upperarm_preroll" />
@@ -266,5 +266,5 @@
       link="upperarm" />
     <axis
-      xyz="0 0 -1" />
+      xyz="0 0 1" />
     <limit
       lower="-1.56"
@@ -295,19 +295,19 @@
       <geometry>
         <mesh
-          filename="package://gummi_base_$(env ROS_GUMMI_BASE)/meshes/j5_Link.stl" />
-      </geometry>
-      <material
-        name="">
-        <color
-          rgba="0.79216 0.81961 0.93333 1" />
-      </material>
-    </visual>
-    <collision>
-      <origin
-        xyz="0 0 0"
-        rpy="0 0 0" />
-      <geometry>
-        <mesh
-          filename="package://gummi_base_$(env ROS_GUMMI_BASE)/meshes/j5_Link.stl" />
+          filename="package://gummi_base_$(env ROS_GUMMI_BASE)/meshes/lowerarm_preroll_u.stl" />
+      </geometry>
+      <material
+        name="">
+        <color
+          rgba="0.79216 0.81961 0.93333 1" />
+      </material>
+    </visual>
+    <collision>
+      <origin
+        xyz="0 0 0"
+        rpy="0 0 0" />
+      <geometry>
+        <mesh
+          filename="package://gummi_base_$(env ROS_GUMMI_BASE)/meshes/lowerarm_preroll_u.stl" />
       </geometry>
     </collision>
@@ -317,6 +317,6 @@
     type="revolute">
     <origin
-      xyz="-0.006 0.0184 -0.23533"
-      rpy="0 0 0" />
+      xyz="-0.0212 0.003 -0.2338"
+      rpy="3.16 1.57 0" />
     <parent
       link="upperarm" />
@@ -324,5 +324,5 @@
       link="lowerarm_preroll_u" />
     <axis
-      xyz="0 -1 0" />
+      xyz="0 0 1" />
     <limit
       lower="-0.75"
@@ -331,5 +331,5 @@
       velocity="0" />
   </joint>
-  <link
+  <!-- <link
     name="upperarm_biceps_pulley">
     <inertial>
@@ -654,4 +654,4 @@
     <axis
       xyz="0 0 0" />
-  </joint>
+  </joint> -->
 </robot>

Commit message: Added Head Functionality
Made the changes that I could see needed to happen to allow me to have a head as a separate package and have it be able to plan and execute through moveit

File: xacro/gummi.srdf.xacro (robot description, xacro)
@@ -17,5 +17,8 @@
     <group name="right_arm">
       <xacro:group_right_arm_base />
-        <xacro:group_right_arm_ee />
+      <xacro:group_right_arm_ee />
+    </group>
+    <group name="head">
+      <xacro:group_head_twodof />
     </group>
     <!--GROUP STATES: Purpose: Define a named state for a particular group, in terms of joint values. This is useful to define states like 'folded arms'-->
@@ -23,4 +26,20 @@
       <xacro:group_state_right_arm_base />
       <xacro:group_state_right_arm_ee />
+    </group_state>
+    <group_state name="default" group="head">
+      <xacro:group_state_head_twodof />
+    </group_state>
+    <group_state name="dab" group="head">
+        <joint name="head_pitch" value="-0.6214" />
+        <joint name="head_yaw" value="-0.5524" />
+    </group_state>
+    <group_state name="dab" group="right_arm">
+        <joint name="elbow" value="-0.75" />
+        <joint name="forearm_roll" value="0.0003" />
+        <joint name="shoulder_pitch" value="0" />
+        <joint name="shoulder_roll" value="1.4787" />
+        <joint name="shoulder_yaw" value="0.5577" />
+        <joint name="upperarm_roll" value="-0.9429" />
+        <joint name="wrist_pitch" value="0" />
     </group_state>
     <xacro:virtual_joints_base />

File: xacro/gummi_description_base.urdf.xacro (robot description, xacro)
@@ -266,5 +266,5 @@
       link="upperarm" />
     <axis
-      xyz="0 0 1" />
+      xyz="0 0 -1" />
     <limit
       lower="-1.56"

Commit message: Added the head and pointer gripper functionality

File: xacro/gummi.srdf.xacro (robot description, xacro)
@@ -22,6 +22,15 @@
       <xacro:group_head_twodof />
     </group>
+    <group name="pointer">
+      <xacro:group_right_arm_base />
+      <xacro:group_right_arm_ee />
+      <xacro:group_pointer />
+    </group>
     <!--GROUP STATES: Purpose: Define a named state for a particular group, in terms of joint values. This is useful to define states like 'folded arms'-->
     <group_state name="default" group="right_arm">
+      <xacro:group_state_right_arm_base />
+      <xacro:group_state_right_arm_ee />
+    </group_state>
+    <group_state name="default" group="pointer">
       <xacro:group_state_right_arm_base />
       <xacro:group_state_right_arm_ee />
@@ -43,4 +52,13 @@
         <joint name="wrist_pitch" value="0" />
     </group_state>
+    <group_state name="start" group="pointer">
+        <joint name="elbow" value="0.1807" />
+        <joint name="forearm_roll" value="0.9648" />
+        <joint name="shoulder_pitch" value="0.9420" />
+        <joint name="shoulder_roll" value="0" />
+        <joint name="shoulder_yaw" value="0" />
+        <joint name="upperarm_roll" value="0" />
+        <joint name="wrist_pitch" value="-0.1538" />
+    </group_state>
     <xacro:virtual_joints_base />
     <xacro:disable_collisions_base />

File: xacro/gummi_base.srdf.xacro (robot description, xacro)
@@ -47,4 +47,14 @@
   <disable_collisions link1="lowerarm_preroll_u" link2="upperarm_preroll" reason="Never" />
   <disable_collisions link1="lowerarm_preroll_u" link2="lowerarm_preroll_d" reason="Adjacent" />
+  <disable_collisions link1="head_pitch" link2="pointer" reason="Never" />
+  <disable_collisions link1="head_yaw" link2="pointer" reason="Never" />
+  <disable_collisions link1="lowerarm" link2="pointer" reason="Never" />
+  <disable_collisions link1="lowerarm_preroll_d" link2="pointer" reason="Never" />
+  <disable_collisions link1="lowerarm_preroll_u" link2="pointer" reason="Never" />
+  <disable_collisions link1="pointer" link2="shoulder" reason="Never" />
+  <disable_collisions link1="pointer" link2="shoulder_preroll" reason="Never" />
+  <disable_collisions link1="pointer" link2="upperarm" reason="Never" />
+  <disable_collisions link1="pointer" link2="upperarm_preroll" reason="Never" />
+  <disable_collisions link1="pointer" link2="wrist" reason="Adjacent" />
 </xacro:macro>
 </robot>

Commit message: rearranged cabling for speed where i want it

File: xacro/gummi.srdf.xacro (robot description, xacro)
@@ -32,6 +32,6 @@
     </group_state>
     <group_state name="dab" group="head">
-        <joint name="head_pitch" value="-0.6214" />
-        <joint name="head_yaw" value="-0.5524" />
+        <joint name="head_pitch" value="-0.6" />
+        <joint name="head_yaw" value="-0.2" />
     </group_state>
     <group_state name="dab" group="right_arm">
