Commit message: Made necessary changes for Luffy

File: xacro/gummi_description_base.urdf.xacro (robot description, xacro)
@@ -3,5 +3,5 @@
   <link
     name="base_link">
-    <inertial>
+    <!-- <inertial>
       <origin
         xyz="-9.81410393552373E-06 -0.0460000689343235 -0.0065295158451983"
@@ -16,12 +16,12 @@
         iyz="-1.48426357415501E-05"
         izz="5.80238931250525E-06" />
-    </inertial>
-    <visual>
-      <origin
-        xyz="0 0 0"
-        rpy="0 0 0" />
-      <geometry>
-        <mesh
-          filename="package://gummi_base_$(env ROS_GUMMI_BASE)/meshes/base_link.STL" />
+    </inertial> -->
+    <visual>
+      <origin
+        xyz="0 0 0"
+        rpy="0 0 0" />
+      <geometry>
+        <mesh
+          filename="package://gummi_base_$(env ROS_GUMMI_BASE)/meshes/base_Link.STL" />
       </geometry>
       <material
@@ -37,5 +37,5 @@
       <geometry>
         <mesh
-          filename="package://gummi_base_$(env ROS_GUMMI_BASE)/meshes/base_link.STL" />
+          filename="package://gummi_base_$(env ROS_GUMMI_BASE)/meshes/base_Link.STL" />
       </geometry>
     </collision>
@@ -63,19 +63,19 @@
       <geometry>
         <mesh
-          filename="package://gummi_base_$(env ROS_GUMMI_BASE)/meshes/shoulder_preroll.STL" />
-      </geometry>
-      <material
-        name="">
-        <color
-          rgba="0.79216 0.81961 0.93333 1" />
-      </material>
-    </visual>
-    <collision>
-      <origin
-        xyz="0 0 0"
-        rpy="0 0 0" />
-      <geometry>
-        <mesh
-          filename="package://gummi_base_$(env ROS_GUMMI_BASE)/meshes/shoulder_preroll.STL" />
+          filename="package://gummi_base_$(env ROS_GUMMI_BASE)/meshes/j1_Link.stl" />
+      </geometry>
+      <material
+        name="">
+        <color
+          rgba="0.79216 0.81961 0.93333 1" />
+      </material>
+    </visual>
+    <collision>
+      <origin
+        xyz="0 0 0"
+        rpy="0 0 0" />
+      <geometry>
+        <mesh
+          filename="package://gummi_base_$(env ROS_GUMMI_BASE)/meshes/j1_Link.stl" />
       </geometry>
     </collision>
@@ -121,19 +121,19 @@
       <geometry>
         <mesh
-          filename="package://gummi_base_$(env ROS_GUMMI_BASE)/meshes/shoulder.STL" />
-      </geometry>
-      <material
-        name="">
-        <color
-          rgba="0.79216 0.81961 0.93333 1" />
-      </material>
-    </visual>
-    <collision>
-      <origin
-        xyz="0 0 0"
-        rpy="0 0 0" />
-      <geometry>
-        <mesh
-          filename="package://gummi_base_$(env ROS_GUMMI_BASE)/meshes/shoulder.STL" />
+          filename="package://gummi_base_$(env ROS_GUMMI_BASE)/meshes/j2_Link.stl" />
+      </geometry>
+      <material
+        name="">
+        <color
+          rgba="0.79216 0.81961 0.93333 1" />
+      </material>
+    </visual>
+    <collision>
+      <origin
+        xyz="0 0 0"
+        rpy="0 0 0" />
+      <geometry>
+        <mesh
+          filename="package://gummi_base_$(env ROS_GUMMI_BASE)/meshes/j2_Link.stl" />
       </geometry>
     </collision>
@@ -179,19 +179,19 @@
       <geometry>
         <mesh
-          filename="package://gummi_base_$(env ROS_GUMMI_BASE)/meshes/upperarm_preroll.STL" />
-      </geometry>
-      <material
-        name="">
-        <color
-          rgba="0.79216 0.81961 0.93333 1" />
-      </material>
-    </visual>
-    <collision>
-      <origin
-        xyz="0 0 0"
-        rpy="0 0 0" />
-      <geometry>
-        <mesh
-          filename="package://gummi_base_$(env ROS_GUMMI_BASE)/meshes/upperarm_preroll.STL" />
+          filename="package://gummi_base_$(env ROS_GUMMI_BASE)/meshes/j3_Link.stl" />
+      </geometry>
+      <material
+        name="">
+        <color
+          rgba="0.79216 0.81961 0.93333 1" />
+      </material>
+    </visual>
+    <collision>
+      <origin
+        xyz="0 0 0"
+        rpy="0 0 0" />
+      <geometry>
+        <mesh
+          filename="package://gummi_base_$(env ROS_GUMMI_BASE)/meshes/j3_Link.stl" />
       </geometry>
     </collision>
@@ -237,19 +237,19 @@
       <geometry>
         <mesh
-          filename="package://gummi_base_$(env ROS_GUMMI_BASE)/meshes/upperarm.STL" />
-      </geometry>
-      <material
-        name="">
-        <color
-          rgba="0.79216 0.81961 0.93333 1" />
-      </material>
-    </visual>
-    <collision>
-      <origin
-        xyz="0 0 0"
-        rpy="0 0 0" />
-      <geometry>
-        <mesh
-          filename="package://gummi_base_$(env ROS_GUMMI_BASE)/meshes/upperarm.STL" />
+          filename="package://gummi_base_$(env ROS_GUMMI_BASE)/meshes/j4_Link.stl" />
+      </geometry>
+      <material
+        name="">
+        <color
+          rgba="0.79216 0.81961 0.93333 1" />
+      </material>
+    </visual>
+    <collision>
+      <origin
+        xyz="0 0 0"
+        rpy="0 0 0" />
+      <geometry>
+        <mesh
+          filename="package://gummi_base_$(env ROS_GUMMI_BASE)/meshes/j4_Link.stl" />
       </geometry>
     </collision>
@@ -295,19 +295,19 @@
       <geometry>
         <mesh
-          filename="package://gummi_base_$(env ROS_GUMMI_BASE)/meshes/lowerarm_preroll_u.STL" />
-      </geometry>
-      <material
-        name="">
-        <color
-          rgba="0.79216 0.81961 0.93333 1" />
-      </material>
-    </visual>
-    <collision>
-      <origin
-        xyz="0 0 0"
-        rpy="0 0 0" />
-      <geometry>
-        <mesh
-          filename="package://gummi_base_$(env ROS_GUMMI_BASE)/meshes/lowerarm_preroll_u.STL" />
+          filename="package://gummi_base_$(env ROS_GUMMI_BASE)/meshes/j5_Link.stl" />
+      </geometry>
+      <material
+        name="">
+        <color
+          rgba="0.79216 0.81961 0.93333 1" />
+      </material>
+    </visual>
+    <collision>
+      <origin
+        xyz="0 0 0"
+        rpy="0 0 0" />
+      <geometry>
+        <mesh
+          filename="package://gummi_base_$(env ROS_GUMMI_BASE)/meshes/j5_Link.stl" />
       </geometry>
     </collision>

Commit message: Latest version minor changes

File: xacro/gummi_description_base.urdf.xacro (robot description, xacro)
@@ -331,327 +331,3 @@
       velocity="0" />
   </joint>
-  <!-- <link
-    name="upperarm_biceps_pulley">
-    <inertial>
-      <origin
-        xyz="-0.0093595 8.3904E-05 3.1839E-09"
-        rpy="0 0 0" />
-      <mass
-        value="0.01522" />
-      <inertia
-        ixx="4.2234E-11"
-        ixy="3.7608E-09"
-        ixz="-3.5118E-13"
-        iyy="3.3488E-07"
-        iyz="3.9438E-15"
-        izz="3.3492E-07" />
-    </inertial>
-    <visual>
-      <origin
-        xyz="0 0 0"
-        rpy="0 0 0" />
-      <geometry>
-        <mesh
-          filename="package://gummi_base_$(env ROS_GUMMI_BASE)/meshes/upperarm_biceps_pulley.STL" />
-      </geometry>
-      <material
-        name="">
-        <color
-          rgba="0.79216 0.81961 0.93333 1" />
-      </material>
-    </visual>
-    <collision>
-      <origin
-        xyz="0 0 0"
-        rpy="0 0 0" />
-      <geometry>
-        <mesh
-          filename="package://gummi_base_$(env ROS_GUMMI_BASE)/meshes/upperarm_biceps_pulley.STL" />
-      </geometry>
-    </collision>
-  </link>
-  <joint
-    name="upperarm_biceps_pulley_joint"
-    type="fixed">
-    <origin
-      xyz="0.0375 0 -0.10243"
-      rpy="0 0 0" />
-    <parent
-      link="upperarm" />
-    <child
-      link="upperarm_biceps_pulley" />
-    <axis
-      xyz="0 0 0" />
-  </joint>
-  <link
-    name="upperarm_triceps_pulley">
-    <inertial>
-      <origin
-        xyz="0.0093595 8.3904E-05 -3.1839E-09"
-        rpy="0 0 0" />
-      <mass
-        value="0.01522" />
-      <inertia
-        ixx="4.2234E-11"
-        ixy="-3.7608E-09"
-        ixz="-3.5118E-13"
-        iyy="3.3488E-07"
-        iyz="-3.9438E-15"
-        izz="3.3492E-07" />
-    </inertial>
-    <visual>
-      <origin
-        xyz="0 0 0"
-        rpy="0 0 0" />
-      <geometry>
-        <mesh
-          filename="package://gummi_base_$(env ROS_GUMMI_BASE)/meshes/upperarm_triceps_pulley.STL" />
-      </geometry>
-      <material
-        name="">
-        <color
-          rgba="0.79216 0.81961 0.93333 1" />
-      </material>
-    </visual>
-    <collision>
-      <origin
-        xyz="0 0 0"
-        rpy="0 0 0" />
-      <geometry>
-        <mesh
-          filename="package://gummi_base_$(env ROS_GUMMI_BASE)/meshes/upperarm_triceps_pulley.STL" />
-      </geometry>
-    </collision>
-  </link>
-  <joint
-    name="upperarm_triceps_pulley_joint"
-    type="fixed">
-    <origin
-      xyz="-0.0435 0 -0.12843"
-      rpy="0 0 0" />
-    <parent
-      link="upperarm" />
-    <child
-      link="upperarm_triceps_pulley" />
-    <axis
-      xyz="-1 0 0" />
-    <limit
-      effort="0"
-      velocity="0" />
-  </joint>
-  <link
-    name="shoulder_roll_top_pulley">
-    <inertial>
-      <origin
-        xyz="-8.3904E-05 -3.1839E-09 -0.0093595"
-        rpy="0 0 0" />
-      <mass
-        value="0.01522" />
-      <inertia
-        ixx="3.3488E-07"
-        ixy="3.9438E-15"
-        ixz="-3.7608E-09"
-        iyy="3.3492E-07"
-        iyz="3.5118E-13"
-        izz="4.2234E-11" />
-    </inertial>
-    <visual>
-      <origin
-        xyz="0 0 0"
-        rpy="0 0 0" />
-      <geometry>
-        <mesh
-          filename="package://gummi_base_$(env ROS_GUMMI_BASE)/meshes/shoulder_roll_top_pulley.STL" />
-      </geometry>
-      <material
-        name="">
-        <color
-          rgba="0.79216 0.81961 0.93333 1" />
-      </material>
-    </visual>
-    <collision>
-      <origin
-        xyz="0 0 0"
-        rpy="0 0 0" />
-      <geometry>
-        <mesh
-          filename="package://gummi_base_$(env ROS_GUMMI_BASE)/meshes/shoulder_roll_top_pulley.STL" />
-      </geometry>
-    </collision>
-  </link>
-  <joint
-    name="shoulder_roll_top_pulley_joint"
-    type="fixed">
-    <origin
-      xyz="0.0208 -0.06848 0.043"
-      rpy="0 0 0" />
-    <parent
-      link="shoulder" />
-    <child
-      link="shoulder_roll_top_pulley" />
-    <axis
-      xyz="0 0 0" />
-  </joint>
-  <link
-    name="shoulder_roll_bottom_pulley">
-    <inertial>
-      <origin
-        xyz="8.3904E-05 -3.1839E-09 0.0093595"
-        rpy="0 0 0" />
-      <mass
-        value="0.01522" />
-      <inertia
-        ixx="3.3488E-07"
-        ixy="-3.9438E-15"
-        ixz="-3.7608E-09"
-        iyy="3.3492E-07"
-        iyz="-3.5118E-13"
-        izz="4.2234E-11" />
-    </inertial>
-    <visual>
-      <origin
-        xyz="0 0 0"
-        rpy="0 0 0" />
-      <geometry>
-        <mesh
-          filename="package://gummi_base_$(env ROS_GUMMI_BASE)/meshes/shoulder_roll_bottom_pulley.STL" />
-      </geometry>
-      <material
-        name="">
-        <color
-          rgba="0.79216 0.81961 0.93333 1" />
-      </material>
-    </visual>
-    <collision>
-      <origin
-        xyz="0 0 0"
-        rpy="0 0 0" />
-      <geometry>
-        <mesh
-          filename="package://gummi_base_$(env ROS_GUMMI_BASE)/meshes/shoulder_roll_bottom_pulley.STL" />
-      </geometry>
-    </collision>
-  </link>
-  <joint
-    name="shoulder_roll_bottom_pulley"
-    type="fixed">
-    <origin
-      xyz="-0.0208 -0.06848 -0.043"
-      rpy="0 0 0" />
-    <parent
-      link="shoulder" />
-    <child
-      link="shoulder_roll_bottom_pulley" />
-    <axis
-      xyz="0 0 -1" />
-    <limit
-      effort="0"
-      velocity="0" />
-  </joint>
-  <link
-    name="shoulder_pitch_front_pulley">
-    <inertial>
-      <origin
-        xyz="-0.0087313 -9.2787E-11 -0.00016773"
-        rpy="0 0 0" />
-      <mass
-        value="0.027251" />
-      <inertia
-        ixx="2.8324E-10"
-        ixy="-6.4973E-15"
-        ixz="-1.1745E-08"
-        iyy="4.8733E-07"
-        iyz="-1.5668E-16"
-        izz="4.8705E-07" />
-    </inertial>
-    <visual>
-      <origin
-        xyz="0 0 0"
-        rpy="0 0 0" />
-      <geometry>
-        <mesh
-          filename="package://gummi_base_$(env ROS_GUMMI_BASE)/meshes/shoulder_pitch_front_pulley.STL" />
-      </geometry>
-      <material
-        name="">
-        <color
-          rgba="0.79216 0.81961 0.93333 1" />
-      </material>
-    </visual>
-    <collision>
-      <origin
-        xyz="0 0 0"
-        rpy="0 0 0" />
-      <geometry>
-        <mesh
-          filename="package://gummi_base_$(env ROS_GUMMI_BASE)/meshes/shoulder_pitch_front_pulley.STL" />
-      </geometry>
-    </collision>
-  </link>
-  <joint
-    name="shoulder_pitch_pulley_front_joint"
-    type="fixed">
-    <origin
-      xyz="0.067474 -0.024095 0.044"
-      rpy="0 0 0" />
-    <parent
-      link="shoulder_preroll" />
-    <child
-      link="shoulder_pitch_front_pulley" />
-    <axis
-      xyz="0 0 0" />
-  </joint>
-  <link
-    name="shoulder_pitch_back_pulley">
-    <inertial>
-      <origin
-        xyz="0.0087313 9.2787E-11 -0.00016773"
-        rpy="0 0 0" />
-      <mass
-        value="0.027251" />
-      <inertia
-        ixx="2.8324E-10"
-        ixy="-6.4973E-15"
-        ixz="1.1745E-08"
-        iyy="4.8733E-07"
-        iyz="1.5668E-16"
-        izz="4.8705E-07" />
-    </inertial>
-    <visual>
-      <origin
-        xyz="0 0 0"
-        rpy="0 0 0" />
-      <geometry>
-        <mesh
-          filename="package://gummi_base_$(env ROS_GUMMI_BASE)/meshes/shoulder_pitch_back_pulley.STL" />
-      </geometry>
-      <material
-        name="">
-        <color
-          rgba="0.79216 0.81961 0.93333 1" />
-      </material>
-    </visual>
-    <collision>
-      <origin
-        xyz="0 0 0"
-        rpy="0 0 0" />
-      <geometry>
-        <mesh
-          filename="package://gummi_base_$(env ROS_GUMMI_BASE)/meshes/shoulder_pitch_back_pulley.STL" />
-      </geometry>
-    </collision>
-  </link>
-  <joint
-    name="shoulder_pitch_back_pulley_joint"
-    type="fixed">
-    <origin
-      xyz="-0.067526 -0.024095 0.044"
-      rpy="0 0 0" />
-    <parent
-      link="shoulder_preroll" />
-    <child
-      link="shoulder_pitch_back_pulley" />
-    <axis
-      xyz="0 0 0" />
-  </joint> -->
 </robot>
